Commit message: feat:gazebo中可以使用ros2 control了

File: src/resources/robots/COD-2026RoboMaster-Balance/urdf/gazebo.xacro (robot description, xacro)
@@ -2,5 +2,4 @@
 <robot xmlns:xacro="http://www.ros.org/wiki/xacro">
 <!-- Gazebo配置文件 - 包含所有Gazebo特定的配置 -->
-<!-- 此文件通过xacro:include被包含在主xacro文件中 -->
 <!-- Gazebo材质定义 - 匹配MuJoCo中的颜色 -->
 <gazebo reference="base_link">
@@ -51,5 +50,5 @@
 <!-- Gazebo标签用于支持闭链机构仿真 -->
 <gazebo>
-  <!-- 左侧五连杆闭环约束1: 连接Left_front_child2_link和Left_rear_link -->
+  <!-- 左侧五连杆闭环约束1 连接Left_front_child2_link和Left_rear_link -->
   <joint name='Left_loop1_joint' type='revolute'>
     <pose relative_to='Left_rear_link'>-0.1005 -0.025 -0.0035 0 0 0</pose>
@@ -70,5 +69,5 @@
     </axis>
   </joint>
-  <!-- 左侧五连杆闭环约束2: 连接Left_front_child3_link和Left_rear_child1_link -->
+  <!-- 左侧五连杆闭环约束2 连接Left_front_child3_link和Left_rear_child1_link -->
   <joint name='Left_loop2_joint' type='revolute'>
     <pose relative_to='Left_rear_child1_link'>-0.038 0 0.05 0 0 0</pose>
@@ -89,5 +88,5 @@
     </axis>
   </joint>
-  <!-- 右侧五连杆闭环约束1: 连接Right_front_child2_link和Right_rear_link -->
+  <!-- 右侧五连杆闭环约束1 连接Right_front_child2_link和Right_rear_link -->
   <joint name='Right_loop1_joint' type='revolute'>
     <pose relative_to='Right_rear_link'>-0.1 0.0225 -0.008 0 0 0</pose>
@@ -108,5 +107,5 @@
     </axis>
   </joint>
-  <!-- 右侧五连杆闭环约束2: 连接Right_front_child3_link和Right_rear_child1_link -->
+  <!-- 右侧五连杆闭环约束2 连接Right_front_child3_link和Right_rear_child1_link -->
   <joint name='Right_loop2_joint' type='revolute'>
     <pose relative_to='Right_rear_child1_link'>-0.035 0 0.05 0 0 0</pose>

File: src/resources/robots/COD-2026RoboMaster-Balance/urdf/ros2_control.xacro (robot description, xacro)
@@ -1,21 +1,51 @@
 <?xml version="1.0"?>
 <robot xmlns:xacro="http://www.ros.org/wiki/xacro">
-    <ros2_control name="CodBalanceHardwareInterface" type="system">
-        <hardware>
-            <plugin>mock_components/GenericSystem</plugin>
-            <param name="calculate_dynamics">true</param>
-        </hardware>
-        <joint name="Left_Wheel_joint">
-            <command_interface name="velocity" />
-            <state_interface name="position" />
-            <state_interface name="velocity" />
-            <state_interface name="effort" />
-        </joint>
-        <joint name="Right_Wheel_joint">
-            <command_interface name="velocity" />
-            <state_interface name="position" />
-            <state_interface name="velocity" />
-            <state_interface name="effort" />
-        </joint>
-    </ros2_control>
+    <xacro:arg name="use_gazebo" default="false"/>
+    <xacro:if value="$(arg use_gazebo)">
+        <!-- Gazebo ROS2 Control Plugin -->
+        <gazebo>
+            <plugin filename="libgazebo_ros2_control.so" name="gazebo_ros2_control">
+                <parameters>$(find bringup)/config/cod_balance_controllers.yaml</parameters>
+            </plugin>
+        </gazebo>
+        <!-- ROS2 Control for Gazebo -->
+        <ros2_control name="CodBalanceHardwareInterface" type="system">
+            <hardware>
+                <plugin>gazebo_ros2_control/GazeboSystem</plugin>
+            </hardware>
+            <joint name="Left_Wheel_joint">
+                <command_interface name="velocity" />
+                <state_interface name="position" />
+                <state_interface name="velocity" />
+                <state_interface name="effort" />
+            </joint>
+            <joint name="Right_Wheel_joint">
+                <command_interface name="velocity" />
+                <state_interface name="position" />
+                <state_interface name="velocity" />
+                <state_interface name="effort" />
+            </joint>
+        </ros2_control>
+    </xacro:if>
+    <xacro:unless value="$(arg use_gazebo)">
+        <!-- ROS2 Control for Real Hardware/Mock -->
+        <ros2_control name="CodBalanceHardwareInterface" type="system">
+            <hardware>
+                <plugin>mock_components/GenericSystem</plugin>
+                <param name="calculate_dynamics">true</param>
+            </hardware>
+            <joint name="Left_Wheel_joint">
+                <command_interface name="velocity" />
+                <state_interface name="position" />
+                <state_interface name="velocity" />
+                <state_interface name="effort" />
+            </joint>
+            <joint name="Right_Wheel_joint">
+                <command_interface name="velocity" />
+                <state_interface name="position" />
+                <state_interface name="velocity" />
+                <state_interface name="effort" />
+            </joint>
+        </ros2_control>
+    </xacro:unless>
 </robot>
