Commit message: feat:vmc控制成功运行 取消皮诺曹求解

File: src/resources/robots/COD-2026RoboMaster-Balance/urdf/ros2_control.xacro (robot description, xacro)
@@ -39,11 +39,11 @@
                 <state_interface name="effort" />
             </joint>
+            <joint name="Right_Wheel_joint">
+                <command_interface name="effort" />
+                <state_interface name="position" />
+                <state_interface name="velocity" />
+                <state_interface name="effort" />
+            </joint>
             <joint name="Right_rear_joint">
-                <command_interface name="effort" />
-                <state_interface name="position" />
-                <state_interface name="velocity" />
-                <state_interface name="effort" />
-            </joint>
-            <joint name="Right_Wheel_joint">
                 <command_interface name="effort" />
                 <state_interface name="position" />
@@ -105,12 +105,12 @@
                 <state_interface name="effort" />
             </joint>
-            <joint name="Right_rear_joint">
-                <command_interface name="effort" />
-                <state_interface name="position" />
-                <state_interface name="velocity" />
-                <state_interface name="effort" />
-            </joint>
             <joint name="Right_Wheel_joint">
                 <command_interface name="velocity" />
+                <command_interface name="effort" />
+                <state_interface name="position" />
+                <state_interface name="velocity" />
+                <state_interface name="effort" />
+            </joint>
+            <joint name="Right_rear_joint">
                 <command_interface name="effort" />
                 <state_interface name="position" />
@@ -181,34 +181,35 @@
                 <param name="model">P1010B_111</param>
                 <param name="can_bus">can1</param>
+                <param name="can_id">0x51</param>
+                <param name="encoder_zero_point">-8191</param>
+                <param name="reduction_ratio">1</param>
+                <param name="reversed">true</param>
+                <param name="multi_turn_angle">false</param>
+            </joint>
+            <!-- Right_Wheel 必须在 Right_rear 之前：二者在 BM 分组帧 0x32 上共用 slot1(motor_id=2)，后写入的覆盖先写入的 -->
+            <joint name="Right_Wheel_joint">
+                <command_interface name="effort" />
+                <state_interface name="position" />
+                <state_interface name="velocity" />
+                <state_interface name="effort" />
+                <param name="vendor">BM</param>
+                <param name="model">M1505B_111</param>
+                <param name="can_bus">can1</param>
+                <param name="can_id">0x0A2</param>
+                <param name="encoder_zero_point">0</param>
+                <param name="reduction_ratio">1</param>
+                <param name="reversed">false</param>
+                <param name="multi_turn_angle">false</param>
+            </joint>
+            <joint name="Right_rear_joint">
+                <command_interface name="effort" />
+                <state_interface name="position" />
+                <state_interface name="velocity" />
+                <state_interface name="effort" />
+                <param name="vendor">BM</param>
+                <param name="model">P1010B_111</param>
+                <param name="can_bus">can1</param>
                 <param name="can_id">0x52</param>
-                <param name="encoder_zero_point">7000</param>
-                <param name="reduction_ratio">1</param>
-                <param name="reversed">false</param>
-                <param name="multi_turn_angle">false</param>
-            </joint>
-            <joint name="Right_rear_joint">
-                <command_interface name="effort" />
-                <state_interface name="position" />
-                <state_interface name="velocity" />
-                <state_interface name="effort" />
-                <param name="vendor">BM</param>
-                <param name="model">P1010B_111</param>
-                <param name="can_bus">can1</param>
-                <param name="can_id">0x51</param>
-                <param name="encoder_zero_point">0</param>
-                <param name="reduction_ratio">1</param>
-                <param name="reversed">false</param>
-                <param name="multi_turn_angle">false</param>
-            </joint>
-            <joint name="Right_Wheel_joint">
-                <command_interface name="effort" />
-                <state_interface name="position" />
-                <state_interface name="velocity" />
-                <state_interface name="effort" />
-                <param name="vendor">BM</param>
-                <param name="model">M1505B_111</param>
-                <param name="can_bus">can1</param>
-                <param name="can_id">0x0A2</param>
-                <param name="encoder_zero_point">0</param>
+                <param name="encoder_zero_point">8191</param>
                 <param name="reduction_ratio">1</param>
                 <param name="reversed">false</param>
