Commit message: feat:添加六个关节的力矩控制 有bug,发送力矩时不是连续的而是反复跳变的

File: src/resources/robots/COD-2026RoboMaster-Balance/urdf/COD_2026_Balance_2_0.xacro (robot description, xacro)
@@ -100,5 +100,5 @@
       lower="0"
       upper="0"
-      effort="0"
+      effort="100"
       velocity="0" />
   </joint>
@@ -332,5 +332,5 @@
       lower="0"
       upper="0"
-      effort="0"
+      effort="100"
       velocity="0" />
   </joint>
@@ -448,5 +448,5 @@
       lower="0"
       upper="0"
-      effort="0"
+      effort="100"
       velocity="0" />
   </joint>
@@ -506,5 +506,5 @@
       lower="0"
       upper="0"
-      effort="0"
+      effort="100"
       velocity="0" />
   </joint>
@@ -738,5 +738,5 @@
       lower="0"
       upper="0"
-      effort="0"
+      effort="100"
       velocity="0" />
   </joint>
@@ -851,4 +851,9 @@
     <axis
       xyz="0 -1 0" />
+    <limit
+      lower="0"
+      upper="0"
+      effort="100"
+      velocity="0" />
   </joint>
 </robot>

File: src/resources/robots/COD-2026RoboMaster-Balance/urdf/gazebo.xacro (robot description, xacro)
@@ -48,4 +48,97 @@
   <material>Gazebo/Grey</material>
 </gazebo>
+<!-- Gazebo关节配置 - 覆盖URDF中的限制，使关节可以受控
+<gazebo reference="Left_front_joint">
+  <implicitSpringDamper>1</implicitSpringDamper>
+  <stopCfm>0.00001</stopCfm>
+  <stopErp>0.1</stopErp>
+  <fudgeFactor>0.5</fudgeFactor>
+  <limit>
+    <lower>-3.14</lower>
+    <upper>3.14</upper>
+    <effort>30</effort>
+    <velocity>10</velocity>
+  </limit>
+  <dynamics>
+    <damping>0.1</damping>
+    <friction>0.01</friction>
+  </dynamics>
+</gazebo>
+<gazebo reference="Left_rear_joint">
+  <implicitSpringDamper>1</implicitSpringDamper>
+  <stopCfm>0.00001</stopCfm>
+  <stopErp>0.1</stopErp>
+  <fudgeFactor>0.5</fudgeFactor>
+  <limit>
+    <lower>-3.14</lower>
+    <upper>3.14</upper>
+    <effort>30</effort>
+    <velocity>10</velocity>
+  </limit>
+  <dynamics>
+    <damping>0.1</damping>
+    <friction>0.01</friction>
+  </dynamics>
+</gazebo>
+<gazebo reference="Left_Wheel_joint">
+  <implicitSpringDamper>1</implicitSpringDamper>
+  <stopCfm>0.00001</stopCfm>
+  <stopErp>0.1</stopErp>
+  <fudgeFactor>0.5</fudgeFactor>
+  <limit>
+    <effort>30</effort>
+    <velocity>100</velocity>
+  </limit>
+  <dynamics>
+    <damping>0.01</damping>
+    <friction>0.01</friction>
+  </dynamics>
+</gazebo>
+<gazebo reference="Right_front_joint">
+  <implicitSpringDamper>1</implicitSpringDamper>
+  <stopCfm>0.00001</stopCfm>
+  <stopErp>0.1</stopErp>
+  <fudgeFactor>0.5</fudgeFactor>
+  <limit>
+    <lower>-3.14</lower>
+    <upper>3.14</upper>
+    <effort>30</effort>
+    <velocity>10</velocity>
+  </limit>
+  <dynamics>
+    <damping>0.1</damping>
+    <friction>0.01</friction>
+  </dynamics>
+</gazebo>
+<gazebo reference="Right_rear_joint">
+  <implicitSpringDamper>1</implicitSpringDamper>
+  <stopCfm>0.00001</stopCfm>
+  <stopErp>0.1</stopErp>
+  <fudgeFactor>0.5</fudgeFactor>
+  <limit>
+    <lower>-3.14</lower>
+    <upper>3.14</upper>
+    <effort>30</effort>
+    <velocity>10</velocity>
+  </limit>
+  <dynamics>
+    <damping>0.1</damping>
+    <friction>0.01</friction>
+  </dynamics>
+</gazebo>
+<gazebo reference="Right_Wheel_joint">
+  <implicitSpringDamper>1</implicitSpringDamper>
+  <stopCfm>0.00001</stopCfm>
+  <stopErp>0.1</stopErp>
+  <fudgeFactor>0.5</fudgeFactor>
+  <limit>
+    <effort>30</effort>
+    <velocity>100</velocity>
+  </limit>
+  <dynamics>
+    <damping>0.01</damping>
+    <friction>0.01</friction>
+  </dynamics>
+</gazebo> -->
 <!-- Gazebo标签用于支持闭链机构仿真 -->
 <gazebo>
@@ -115,6 +208,6 @@
       <xyz>0 -1 0</xyz>
       <limit>
-        <lower>-1.3</lower>
-        <upper>0</upper>
+        <lower>0</lower>
+        <upper>1.3</upper>
         <effort>0</effort>
         <velocity>0</velocity>

File: src/resources/robots/COD-2026RoboMaster-Balance/urdf/ros2_control.xacro (robot description, xacro)
@@ -14,6 +14,31 @@
                 <plugin>gazebo_ros2_control/GazeboSystem</plugin>
             </hardware>
+            <joint name="Left_front_joint">
+                <command_interface name="effort" />
+                <state_interface name="position" />
+                <state_interface name="velocity" />
+                <state_interface name="effort" />
+            </joint>
+            <joint name="Left_rear_joint">
+                <command_interface name="effort" />
+                <state_interface name="position" />
+                <state_interface name="velocity" />
+                <state_interface name="effort" />
+            </joint>
             <joint name="Left_Wheel_joint">
                 <command_interface name="velocity" />
+                <command_interface name="effort" />
+                <state_interface name="position" />
+                <state_interface name="velocity" />
+                <state_interface name="effort" />
+            </joint>
+            <joint name="Right_front_joint">
+                <command_interface name="effort" />
+                <state_interface name="position" />
+                <state_interface name="velocity" />
+                <state_interface name="effort" />
+            </joint>
+            <joint name="Right_rear_joint">
+                <command_interface name="effort" />
                 <state_interface name="position" />
                 <state_interface name="velocity" />
@@ -22,4 +47,5 @@
             <joint name="Right_Wheel_joint">
                 <command_interface name="velocity" />
+                <command_interface name="effort" />
                 <state_interface name="position" />
                 <state_interface name="velocity" />
@@ -35,6 +61,31 @@
                 <param name="calculate_dynamics">true</param>
             </hardware>
+            <joint name="Left_front_joint">
+                <command_interface name="effort" />
+                <state_interface name="position" />
+                <state_interface name="velocity" />
+                <state_interface name="effort" />
+            </joint>
+            <joint name="Left_rear_joint">
+                <command_interface name="effort" />
+                <state_interface name="position" />
+                <state_interface name="velocity" />
+                <state_interface name="effort" />
+            </joint>
             <joint name="Left_Wheel_joint">
                 <command_interface name="velocity" />
+                <command_interface name="effort" />
+                <state_interface name="position" />
+                <state_interface name="velocity" />
+                <state_interface name="effort" />
+            </joint>
+            <joint name="Right_front_joint">
+                <command_interface name="effort" />
+                <state_interface name="position" />
+                <state_interface name="velocity" />
+                <state_interface name="effort" />
+            </joint>
+            <joint name="Right_rear_joint">
+                <command_interface name="effort" />
                 <state_interface name="position" />
                 <state_interface name="velocity" />
@@ -43,4 +94,5 @@
             <joint name="Right_Wheel_joint">
                 <command_interface name="velocity" />
+                <command_interface name="effort" />
                 <state_interface name="position" />
                 <state_interface name="velocity" />

Commit message: update:添加m控制器，准备验证

File: src/resources/robots/COD-2026RoboMaster-Balance/urdf/COD_2026_Balance_2_0.xacro (robot description, xacro)
@@ -101,5 +101,5 @@
       upper="0"
       effort="100"
-      velocity="0" />
+      velocity="100" />
   </joint>
   <link
@@ -333,5 +333,5 @@
       upper="0"
       effort="100"
-      velocity="0" />
+      velocity="100" />
   </joint>
   <link
@@ -449,5 +449,5 @@
       upper="0"
       effort="100"
-      velocity="0" />
+      velocity="100" />
   </joint>
   <link
@@ -507,5 +507,5 @@
       upper="0"
       effort="100"
-      velocity="0" />
+      velocity="100" />
   </joint>
   <link
@@ -739,5 +739,5 @@
       upper="0"
       effort="100"
-      velocity="0" />
+      velocity="100" />
   </joint>
   <link
@@ -855,5 +855,5 @@
       upper="0"
       effort="100"
-      velocity="0" />
+      velocity="100" />
   </joint>
 </robot>

File: src/resources/robots/COD-2026RoboMaster-Balance/urdf/gazebo.xacro (robot description, xacro)
@@ -48,5 +48,6 @@
   <material>Gazebo/Grey</material>
 </gazebo>
-<!-- Gazebo关节配置 - 覆盖URDF中的限制，使关节可以受控
+<!-- Gazebo关节配置 - 包含关节摩擦力和动力学参数 -->
+<!-- 左侧前腿关节 -->
 <gazebo reference="Left_front_joint">
   <implicitSpringDamper>1</implicitSpringDamper>
@@ -62,7 +63,56 @@
   <dynamics>
     <damping>0.1</damping>
-    <friction>0.01</friction>
-  </dynamics>
-</gazebo>
+    <friction>0.1</friction>
+  </dynamics>
+</gazebo>
+<gazebo reference="Left_front_child1_joint">
+  <implicitSpringDamper>1</implicitSpringDamper>
+  <stopCfm>0.00001</stopCfm>
+  <stopErp>0.1</stopErp>
+  <fudgeFactor>0.5</fudgeFactor>
+  <limit>
+    <lower>-3.14</lower>
+    <upper>3.14</upper>
+    <effort>30</effort>
+    <velocity>10</velocity>
+  </limit>
+  <dynamics>
+    <damping>0.1</damping>
+    <friction>0.1</friction>
+  </dynamics>
+</gazebo>
+<gazebo reference="Left_front_child2_joint">
+  <implicitSpringDamper>1</implicitSpringDamper>
+  <stopCfm>0.00001</stopCfm>
+  <stopErp>0.1</stopErp>
+  <fudgeFactor>0.5</fudgeFactor>
+  <limit>
+    <lower>-3.14</lower>
+    <upper>3.14</upper>
+    <effort>30</effort>
+    <velocity>10</velocity>
+  </limit>
+  <dynamics>
+    <damping>0.1</damping>
+    <friction>0.1</friction>
+  </dynamics>
+</gazebo>
+<gazebo reference="Left_front_child3_joint">
+  <implicitSpringDamper>1</implicitSpringDamper>
+  <stopCfm>0.00001</stopCfm>
+  <stopErp>0.1</stopErp>
+  <fudgeFactor>0.5</fudgeFactor>
+  <limit>
+    <lower>-3.14</lower>
+    <upper>3.14</upper>
+    <effort>30</effort>
+    <velocity>10</velocity>
+  </limit>
+  <dynamics>
+    <damping>0.1</damping>
+    <friction>0.1</friction>
+  </dynamics>
+</gazebo>
+<!-- 左侧后腿关节 -->
 <gazebo reference="Left_rear_joint">
   <implicitSpringDamper>1</implicitSpringDamper>
@@ -78,7 +128,24 @@
   <dynamics>
     <damping>0.1</damping>
-    <friction>0.01</friction>
-  </dynamics>
-</gazebo>
+    <friction>0.1</friction>
+  </dynamics>
+</gazebo>
+<gazebo reference="Left_rear_child1_joint">
+  <implicitSpringDamper>1</implicitSpringDamper>
+  <stopCfm>0.00001</stopCfm>
+  <stopErp>0.1</stopErp>
+  <fudgeFactor>0.5</fudgeFactor>
+  <limit>
+    <lower>-3.14</lower>
+    <upper>3.14</upper>
+    <effort>30</effort>
+    <velocity>10</velocity>
+  </limit>
+  <dynamics>
+    <damping>0.1</damping>
+    <friction>0.1</friction>
+  </dynamics>
+</gazebo>
+<!-- 左侧轮子关节 -->
 <gazebo reference="Left_Wheel_joint">
   <implicitSpringDamper>1</implicitSpringDamper>
@@ -92,7 +159,8 @@
   <dynamics>
     <damping>0.01</damping>
-    <friction>0.01</friction>
-  </dynamics>
-</gazebo>
+    <friction>0.1</friction>
+  </dynamics>
+</gazebo>
+<!-- 右侧前腿关节 -->
 <gazebo reference="Right_front_joint">
   <implicitSpringDamper>1</implicitSpringDamper>
@@ -108,7 +176,56 @@
   <dynamics>
     <damping>0.1</damping>
-    <friction>0.01</friction>
-  </dynamics>
-</gazebo>
+    <friction>0.1</friction>
+  </dynamics>
+</gazebo>
+<gazebo reference="Right_front_child1_joint">
+  <implicitSpringDamper>1</implicitSpringDamper>
+  <stopCfm>0.00001</stopCfm>
+  <stopErp>0.1</stopErp>
+  <fudgeFactor>0.5</fudgeFactor>
+  <limit>
+    <lower>-3.14</lower>
+    <upper>3.14</upper>
+    <effort>30</effort>
+    <velocity>10</velocity>
+  </limit>
+  <dynamics>
+    <damping>0.1</damping>
+    <friction>0.1</friction>
+  </dynamics>
+</gazebo>
+<gazebo reference="Right_front_child2_joint">
+  <implicitSpringDamper>1</implicitSpringDamper>
+  <stopCfm>0.00001</stopCfm>
+  <stopErp>0.1</stopErp>
+  <fudgeFactor>0.5</fudgeFactor>
+  <limit>
+    <lower>-3.14</lower>
+    <upper>3.14</upper>
+    <effort>30</effort>
+    <velocity>10</velocity>
+  </limit>
+  <dynamics>
+    <damping>0.1</damping>
+    <friction>0.1</friction>
+  </dynamics>
+</gazebo>
+<gazebo reference="Right_front_joint3_joint">
+  <implicitSpringDamper>1</implicitSpringDamper>
+  <stopCfm>0.00001</stopCfm>
+  <stopErp>0.1</stopErp>
+  <fudgeFactor>0.5</fudgeFactor>
+  <limit>
+    <lower>-3.14</lower>
+    <upper>3.14</upper>
+    <effort>30</effort>
+    <velocity>10</velocity>
+  </limit>
+  <dynamics>
+    <damping>0.1</damping>
+    <friction>0.1</friction>
+  </dynamics>
+</gazebo>
+<!-- 右侧后腿关节 -->
 <gazebo reference="Right_rear_joint">
   <implicitSpringDamper>1</implicitSpringDamper>
@@ -124,7 +241,24 @@
   <dynamics>
     <damping>0.1</damping>
-    <friction>0.01</friction>
-  </dynamics>
-</gazebo>
+    <friction>0.1</friction>
+  </dynamics>
+</gazebo>
+<gazebo reference="Right_rear_child1_joint">
+  <implicitSpringDamper>1</implicitSpringDamper>
+  <stopCfm>0.00001</stopCfm>
+  <stopErp>0.1</stopErp>
+  <fudgeFactor>0.5</fudgeFactor>
+  <limit>
+    <lower>-3.14</lower>
+    <upper>3.14</upper>
+    <effort>30</effort>
+    <velocity>10</velocity>
+  </limit>
+  <dynamics>
+    <damping>0.1</damping>
+    <friction>0.1</friction>
+  </dynamics>
+</gazebo>
+<!-- 右侧轮子关节 -->
 <gazebo reference="Right_Wheel_joint">
   <implicitSpringDamper>1</implicitSpringDamper>
@@ -138,7 +272,7 @@
   <dynamics>
     <damping>0.01</damping>
-    <friction>0.01</friction>
-  </dynamics>
-</gazebo> -->
+    <friction>0.1</friction>
+  </dynamics>
+</gazebo>
 <!-- Gazebo标签用于支持闭链机构仿真 -->
 <gazebo>
@@ -157,6 +291,6 @@
       </limit>
       <dynamics>
-        <damping>0.1</damping>
-        <friction>0.01</friction>
+        <damping>0.5</damping>
+        <friction>0.1</friction>
       </dynamics>
     </axis>
@@ -176,6 +310,6 @@
       </limit>
       <dynamics>
-        <damping>0.1</damping>
-        <friction>0.01</friction>
+        <damping>0.5</damping>
+        <friction>0.1</friction>
       </dynamics>
     </axis>
@@ -195,6 +329,6 @@
       </limit>
       <dynamics>
-        <damping>0.1</damping>
-        <friction>0.01</friction>
+        <damping>0.5</damping>
+        <friction>0.1</friction>
       </dynamics>
     </axis>
@@ -214,6 +348,6 @@
       </limit>
       <dynamics>
-        <damping>0.1</damping>
-        <friction>0.01</friction>
+        <damping>0.5</damping>
+        <friction>0.1</friction>
       </dynamics>
     </axis>

File: src/resources/robots/COD-2026RoboMaster-Balance/urdf/ros2_control.xacro (robot description, xacro)
@@ -2,4 +2,5 @@
 <robot xmlns:xacro="http://www.ros.org/wiki/xacro">
     <xacro:arg name="use_gazebo" default="false"/>
+    <xacro:arg name="use_mujoco" default="false"/>
     <xacro:if value="$(arg use_gazebo)">
         <!-- Gazebo ROS2 Control Plugin -->
@@ -55,10 +56,10 @@
     </xacro:if>
     <xacro:unless value="$(arg use_gazebo)">
-        <!-- ROS2 Control for Real Hardware/Mock -->
-        <ros2_control name="CodBalanceHardwareInterface" type="system">
-            <hardware>
-                <plugin>mock_components/GenericSystem</plugin>
-                <param name="calculate_dynamics">true</param>
-            </hardware>
+        <xacro:if value="$(arg use_mujoco)">
+            <!-- ROS2 Control for MuJoCo -->
+            <ros2_control name="MujocoSystem" type="system">
+                <hardware>
+                    <plugin>mujoco_ros2_control/MujocoSystem</plugin>
+                </hardware>
             <joint name="Left_front_joint">
                 <command_interface name="effort" />
@@ -100,4 +101,52 @@
             </joint>
         </ros2_control>
+        </xacro:if>
+        <xacro:unless value="$(arg use_mujoco)">
+            <!-- ROS2 Control for Real Hardware/Mock -->
+            <ros2_control name="CodBalanceHardwareInterface" type="system">
+                <hardware>
+                    <plugin>mock_components/GenericSystem</plugin>
+                    <param name="calculate_dynamics">true</param>
+                </hardware>
+            <joint name="Left_front_joint">
+                <command_interface name="effort" />
+                <state_interface name="position" />
+                <state_interface name="velocity" />
+                <state_interface name="effort" />
+            </joint>
+            <joint name="Left_rear_joint">
+                <command_interface name="effort" />
+                <state_interface name="position" />
+                <state_interface name="velocity" />
+                <state_interface name="effort" />
+            </joint>
+            <joint name="Left_Wheel_joint">
+                <command_interface name="velocity" />
+                <command_interface name="effort" />
+                <state_interface name="position" />
+                <state_interface name="velocity" />
+                <state_interface name="effort" />
+            </joint>
+            <joint name="Right_front_joint">
+                <command_interface name="effort" />
+                <state_interface name="position" />
+                <state_interface name="velocity" />
+                <state_interface name="effort" />
+            </joint>
+            <joint name="Right_rear_joint">
+                <command_interface name="effort" />
+                <state_interface name="position" />
+                <state_interface name="velocity" />
+                <state_interface name="effort" />
+            </joint>
+            <joint name="Right_Wheel_joint">
+                <command_interface name="velocity" />
+                <command_interface name="effort" />
+                <state_interface name="position" />
+                <state_interface name="velocity" />
+                <state_interface name="effort" />
+            </joint>
+        </ros2_control>
+        </xacro:unless>
     </xacro:unless>
 </robot>

Commit message: feat:加入real imu

File: src/resources/robots/COD-2026RoboMaster-Balance/urdf/COD_2026_Balance_2_0.xacro (robot description, xacro)
@@ -45,4 +45,10 @@
     </collision>
   </link>
+  <link name="imu_link"/>
+  <joint name="imu_joint" type="fixed">
+    <origin xyz="0 0 0" rpy="0 0 0" />
+    <parent link="base_link" />
+    <child link="imu_link" />
+  </joint>
   <link
     name="Left_front_link">

File: src/resources/robots/COD-2026RoboMaster-Balance/urdf/cod_balance_simple.xacro (robot description, xacro)
@@ -22,4 +22,10 @@
     </collision>
   </link>
+  <link name="imu_link"/>
+  <joint name="imu_joint" type="fixed">
+    <origin xyz="0 0 0" rpy="0 0 0" />
+    <parent link="base_link" />
+    <child link="imu_link" />
+  </joint>
   <link name="Left_rear_link">
     <inertial>

File: src/resources/robots/COD-2026RoboMaster-Balance/urdf/ros2_control.xacro (robot description, xacro)
@@ -130,4 +130,12 @@
                 <param name="command_timeout_ms">100</param>
                 <param name="allow_partial_feedback">true</param>
+                <param name="imu_sensor_name">imu_sensor</param>
+                <param name="imu_sample_freq">1000.0</param>
+                <param name="imu_kp">0.2</param>
+                <param name="imu_ki">0.0</param>
+                <param name="imu_gyro_axes">1,2,3</param>
+                <param name="imu_acc_axes">1,2,3</param>
+                <param name="imu_calibration_enable">0</param>
+                <param name="imu_calibration_file">src/hardware/librmcs_hardware/msg/imu_calibration.yaml</param>
             </hardware>
             <joint name="Left_front_joint">
@@ -216,4 +224,16 @@
                 <param name="multi_turn_angle">false</param>
             </joint>
+            <sensor name="imu_sensor">
+                <state_interface name="orientation.x"/>
+                <state_interface name="orientation.y"/>
+                <state_interface name="orientation.z"/>
+                <state_interface name="orientation.w"/>
+                <state_interface name="angular_velocity.x"/>
+                <state_interface name="angular_velocity.y"/>
+                <state_interface name="angular_velocity.z"/>
+                <state_interface name="linear_acceleration.x"/>
+                <state_interface name="linear_acceleration.y"/>
+                <state_interface name="linear_acceleration.z"/>
+            </sensor>
         </ros2_control>
         </xacro:unless>
